File: hardware/pcb/terrascout.kicad_pcb (KiCad board)
At the start: 2 copper layers, 100 x 80 mm, 30 parts, among them J1 JST-XH-2P, J2 JST-XH-2P, J3 JST-XH-4P, J4 JST-XH-4P, J5 PINHD-1x3, J6 PINHD-1x4, J7 JST-XH-2P, J8 PINHD-1x2, SW1 SPDT_SWITCH, U1 ESP32-S3-DevKitC-1, U2 DRV8833PWP, U3 MP1584EN_3A, U4 TP5100_2S

Commit message: feat(hardware): Add full KiCad PCB, Gerber manufacturing package, DRC validation, and passing test suite
Parts:
- added J9: PINHD-1x4, PinHeader_1x04_P2.54mm_Vertical, F.Cu at (55.0, 13.0)
- added R7: 10k, R_0805_2012Metric, F.Cu at (23.0, 22.5)
- added R8: 10k, R_0805_2012Metric, F.Cu at (54.5, 53.0)
Routing:
- net 3V3: track 181.1 -> 228.0 mm
- net TX: track 0.00 -> 14.4 mm
- net RX: track 0.00 -> 14.4 mm
- net GPIO0: track 0.00 -> 2.15 mm
- net EN: track 0.00 -> 2.05 mm
Changed lines of the file:
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@@
     (pad "2" smd rect (at 0.950 0.000) (size 1.000 1.250) (layers ("F.Cu" "F.Mask" "F.Paste")) (net 1 "GND"))
+  )
+  (footprint "PinHeader_1x04_P2.54mm_Vertical" (layer "F.Cu")
+    (at 55.000 13.000 90)
+    (property "Reference" "J9" (at 0 -2.5 0) (layer "F.SilkS") (effects (font (size 1 1) (thickness 0.15))))
+    (property "Value" "PINHD-1x4" (at 0 2.5 0) (layer "F.Fab") (effects (font (size 1 1) (thickness 0.15))))
+    (pad "1" thru_hole rect (at 0.000 -3.810) (size 1.600 1.600) (drill 0.900) (layers ("*.Cu" "*.Mask")) (net 3 "3V3"))
+    (pad "2" thru_hole circle (at 0.000 -1.270) (size 1.600 1.600) (drill 0.900) (layers ("*.Cu" "*.Mask")) (net 46 "TX"))
+    (pad "3" thru_hole circle (at 0.000 1.270) (size 1.600 1.600) (drill 0.900) (layers ("*.Cu" "*.Mask")) (net 43 "RX"))
+    (pad "4" thru_hole circle (at 0.000 3.810) (size 1.600 1.600) (drill 0.900) (layers ("*.Cu" "*.Mask")) (net 1 "GND"))
+  )
+  (footprint "R_0805_2012Metric" (layer "F.Cu")
+    (at 23.000 22.540 0)
+    (property "Reference" "R7" (at 0 -2.5 0) (layer "F.SilkS") (effects (font (size 1 1) (thickness 0.15))))
+    (property "Value" "10k" (at 0 2.5 0) (layer "F.Fab") (effects (font (size 1 1) (thickness 0.15))))
+    (pad "1" smd rect (at -0.950 0.000) (size 1.000 1.250) (layers ("F.Cu" "F.Mask" "F.Paste")) (net 3 "3V3"))
+    (pad "2" smd rect (at 0.950 0.000) (size 1.000 1.250) (layers ("F.Cu" "F.Mask" "F.Paste")) (net 4 "EN"))
+  )
+  (footprint "R_0805_2012Metric" (layer "F.Cu")
+    (at 54.500 53.020 0)
+    (property "Reference" "R8" (at 0 -2.5 0) (layer "F.SilkS") (effects (font (size 1 1) (thickness 0.15))))
+    (property "Value" "10k" (at 0 2.5 0) (layer "F.Fab") (effects (font (size 1 1) (thickness 0.15))))
+    (pad "1" smd rect (at -0.950 0.000) (size 1.000 1.250) (layers ("F.Cu" "F.Mask" "F.Paste")) (net 3 "3V3"))
+    (pad "2" smd rect (at 0.950 0.000) (size 1.000 1.250) (layers ("F.Cu" "F.Mask" "F.Paste")) (net 5 "GPIO0"))
   )
   (footprint "MountingHole:MountingHole_3.2mm_M3_Pad_Via" (layer "F.Cu")
@@
   (segment (start 76.700 40.370) (end 78.550 40.370) (width 0.305) (layer "F.Cu") (net 50))
   (segment (start 78.550 40.370) (end 78.550 42.000) (width 0.305) (layer "F.Cu") (net 50))
+  (segment (start 51.400 22.540) (end 53.000 22.540) (width 0.305) (layer "F.Cu") (net 46))
+  (segment (start 53.000 22.540) (end 53.000 11.730) (width 0.305) (layer "F.Cu") (net 46))
+  (segment (start 53.000 11.730) (end 55.000 11.730) (width 0.305) (layer "F.Cu") (net 46))
+  (segment (start 51.400 25.080) (end 53.500 25.080) (width 0.305) (layer "F.Cu") (net 43))
+  (segment (start 53.500 25.080) (end 53.500 14.270) (width 0.305) (layer "F.Cu") (net 43))
+  (segment (start 53.500 14.270) (end 55.000 14.270) (width 0.305) (layer "F.Cu") (net 43))
+  (segment (start 26.000 22.540) (end 23.950 22.540) (width 0.305) (layer "F.Cu") (net 4))
+  (segment (start 22.050 22.540) (end 21.500 22.540) (width 0.305) (layer "F.Cu") (net 3))
+  (segment (start 21.500 22.540) (end 21.500 20.000) (width 0.305) (layer "F.Cu") (net 3))
+  (segment (start 21.500 20.000) (end 26.000 20.000) (width 0.305) (layer "F.Cu") (net 3))
+  (segment (start 51.400 53.020) (end 53.550 53.020) (width 0.305) (layer "F.Cu") (net 5))
+  (segment (start 55.450 53.020) (end 57.000 53.020) (width 0.305) (layer "F.Cu") (net 3))
+  (segment (start 57.000 53.020) (end 57.000 52.190) (width 0.305) (layer "F.Cu") (net 3))
+  (segment (start 57.000 52.190) (end 69.000 52.190) (width 0.305) (layer "F.Cu") (net 3))
+  (segment (start 55.000 9.190) (end 57.000 9.190) (width 0.305) (layer "F.Cu") (net 3))
+  (segment (start 57.000 9.190) (end 57.000 8.000) (width 0.305) (layer "F.Cu") (net 3))
+  (segment (start 57.000 8.000) (end 78.750 8.000) (width 0.305) (layer "F.Cu") (net 3))
   (via (at 73.100 41.200) (size 0.600) (drill 0.300) (layers "F.Cu" "B.Cu") (net 1))
   (via (at 73.100 42.000) (size 0.600) (drill 0.300) (layers "F.Cu" "B.Cu") (net 1))
